File: Board Designs/UCCS_Senior_Design_2.brd (EAGLE design)
At the start: 38.5 x 30.2 mm, 24 parts

Commit message: Upteenth Revision of Layout
Connections:
- removed net S$81: R25.1
- new net S$85: C857.1, R17.1, R25.1
Routing:
- net S$85: track 0.00 -> 10.4 mm
Changed lines of the file:
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@@
 <signal name="S$34">
-</signal>
-<signal name="S$81">
-<contactref element="R25" pad="1"/>
-<wire x1="31.4912" y1="24.7986" x2="31.5016" y2="25.0882" width="0.4064" layer="1"/>
 </signal>
 <signal name="S$10">
@@
 </polygon>
 </signal>
+<signal name="S$85">
+<contactref element="R17" pad="1"/>
+<contactref element="C857" pad="1"/>
+<wire x1="31.4602" y1="35.1456" x2="31.4912" y2="35.1456" width="0.4064" layer="1"/>
+<wire x1="31.4912" y1="35.1456" x2="31.4912" y2="26.6924" width="0.4064" layer="1"/>
+<contactref element="R25" pad="1"/>
+<wire x1="31.4912" y1="24.7986" x2="31.5016" y2="25.0882" width="0.4064" layer="1"/>
+<wire x1="31.4912" y1="26.6924" x2="31.5016" y2="26.6924" width="0.4064" layer="1"/>
+<wire x1="31.5016" y1="26.6924" x2="31.5016" y2="25.0882" width="0.4064" layer="1"/>
+</signal>
 </signals>
